Commit message: properties and multiple files

File: src/my_robot_description/urdf/my_robot.urdf.xacro (robot description, xacro)
@@ -1,48 +1,5 @@
 <?xml version="1.0"?>
-<robot name="my_root" xmlns:xacro="http://www.ros.org./wiki/xacro">
-	<material name="green">
-		<color rgba="0 0.5 0 1" />
-	</material>
-	<material name="grey">
-		<color rgba="0.5 0.5 0.5 1" />
-	</material>
-	<link name="base_link">
-		<visual>
-			<geometry>
-				<box size="0.6 0.4 0.2" />
-			</geometry>
-			<origin xyz="0 0 0.1" rpy="0 0 0" />
-			<material name="green" />
-		</visual>
-	</link>
-	<link name="left_wheel_link">
-		<visual>
-			<geometry>
-				<cylinder radius="0.1" length="0.05" />
-			</geometry>
-			<origin xyz="0 0 0" rpy="1.57 0 0" />
-			<material name="grey" />
-		</visual>
-	</link>
-	<link name="right_wheel_link">
-		<visual>
-			<geometry>
-				<cylinder radius="0.1" length="0.05" />
-			</geometry>
-			<origin xyz="0 0 0" rpy="1.57 0 0" />
-			<material name="grey" />
-		</visual>
-	</link>
-	<joint name="base_left_wheel_joint" type="continuous">
-		<parent link="base_link" />
-		<child link="left_wheel_link" />
-		<origin xyz="0 0.225 0" rpy="0 0 0" />
-		<axis xyz="0 1 0" />
-	</joint>
-	<joint name="base_right_wheel_joint" type="continuous">
-		<parent link="base_link" />
-		<child link="right_wheel_link" />
-		<origin xyz="0 -0.225 0" rpy="0 0 0" />
-		<axis xyz="0 1 0" />
-	</joint>
+<robot name="my_robot" xmlns:xacro="http://www.ros.org/wiki/xacro">
+    <xacro:include filename="common_properties.xacro" />
+    <xacro:include filename="mobile_base.xacro" />
 </robot>
