Commit message: fix to work with opencv

File: src/my_robot_description/urdf/camera.xacro (robot description, xacro)
@@ -27,4 +27,11 @@
 		<child link="camera_link" />
 	</joint>
+	<!-- new joint and link to work with opencv -->
+	<joint name="camera_optical_joint" type="fixed">
+		<origin xyz="0 0 0" rpy="${-pi/2} 0 ${-pi/2}" />
+		<parent link="camera_link" />
+		<child link="camera_link_optical" />
+	</joint>
+	<link name="camera_link_optical" />
 	<gazebo reference="camera_link">
 		<material>Gazebo/Red</material>
@@ -34,5 +41,5 @@
 			<update_rate>10.0</update_rate>
 			<plugin name="camera_controller" filename="libgazebo_ros_camera.so">
-				<frame_name>camera_link</frame_name>
+				<frame_name>camera_link_optical</frame_name>
 			</plugin>
 		</sensor>
