Commit message: add inertia

File: src/my_robot_description/urdf/common_properties.xacro (robot description, xacro)
@@ -7,3 +7,30 @@
         <color rgba="0.5 0.5 0.5 1" />
     </material>
+    <xacro:macro name="box_inertia" params="mass length width height xyz rpy">
+        <inertial>
+            <origin xyz="${xyz}" rpy="${rpy}" />
+            <mass value="${mass}" />
+            <inertia ixx="${mass * (length**2 + height**2) / 12.0}" ixy="0.0" ixz="0.0"
+                iyy="${mass * (length**2 + width**2) / 12.0}" iyz="0.0"
+                izz="${mass * (height**2 + width**2) / 12.0}" />
+        </inertial>
+    </xacro:macro>
+    <xacro:macro name="cylinder_inertia" params="mass radius height xyz rpy">
+        <inertial>
+            <origin xyz="${xyz}" rpy="${rpy}" />
+            <mass value="${mass}" />
+            <inertia ixx="${mass * (3 * radius**2 + height**2) / 12.0}" ixy="0.0" ixz="0.0"
+                iyy="${mass * (3 * radius**2 + height**2) / 12.0}" iyz="0.0"
+                izz="${mass * radius**2 / 2.0}" />
+        </inertial>
+    </xacro:macro>
+    <xacro:macro name="sphere_inertia" params="massa radius xyz rpy">
+        <inertial>
+            <origin xyz="${xyz}" rpy="${rpy}" />
+            <mass value="${mass}" />
+            <inertia ixx="${mass * (2 * radius**2) / 5.0}" ixy="0.0" ixz="0.0"
+                iyy="${mass * (2 * radius**2) / 5.0}" iyz="0.0"
+                izz="${mass * (2 * radius**2) / 5.0}" />
+        </inertial>
+    </xacro:macro>
 </robot>

File: src/my_robot_description/urdf/mobile_base.xacro (robot description, xacro)
@@ -15,4 +15,6 @@
             <material name="blue" />
         </visual>
+        <xacro:box_inertia mass="5.0" length="${base_length}" width="${base_width}"
+            height="${base_height}" xyz="0 0 ${base_height / 2.0}" rpy="0 0 0" />
     </link>
     <xacro:macro name="wheel_link" params="prefix">
@@ -26,4 +28,6 @@
             </visual>
         </link>
+        <xacro:cylinder_inertia mass="1.0" radius="${wheel_radius}" height="${wheel_length}"
+            xyz="0 0 0" rpy="${pi / 2.0} 0 0" />
     </xacro:macro>
     <xacro:wheel_link prefix="right" />
@@ -37,9 +41,10 @@
             <material name="grey" />
         </visual>
+        <xacro:sphere_inertia mass="0.5" radius="${wheel_radius / 2.0}" xyz="0 0 0" rpy="0 0 0" />
     </link>
     <joint name="base_joint" type="fixed">
         <parent link="base_footprint" />
         <child link="base_link" />
-        <origin xyz="0 0 ${wheel_radius}" rpy="0 0 0"/>
+        <origin xyz="0 0 ${wheel_radius}" rpy="0 0 0" />
     </joint>
     <joint name="base_right_wheel_joint" type="continuous">

Commit message: add collision

File: src/my_robot_description/urdf/common_properties.xacro (robot description, xacro)
@@ -25,5 +25,5 @@
         </inertial>
     </xacro:macro>
-    <xacro:macro name="sphere_inertia" params="massa radius xyz rpy">
+    <xacro:macro name="sphere_inertia" params="mass radius xyz rpy">
         <inertial>
             <origin xyz="${xyz}" rpy="${rpy}" />

File: src/my_robot_description/urdf/mobile_base.xacro (robot description, xacro)
@@ -15,4 +15,10 @@
             <material name="blue" />
         </visual>
+        <collision>
+            <geometry>
+                <box size="${base_length} ${base_width} ${base_height}" />
+            </geometry>
+            <origin xyz="0 0 ${base_height / 2.0}" rpy="0 0 0" />
+        </collision>
         <xacro:box_inertia mass="5.0" length="${base_length}" width="${base_width}"
             height="${base_height}" xyz="0 0 ${base_height / 2.0}" rpy="0 0 0" />
@@ -27,7 +33,13 @@
                 <material name="grey" />
             </visual>
+            <collision>
+                <geometry>
+                    <cylinder radius="${wheel_radius}" length="${wheel_length}" />
+                </geometry>
+                <origin xyz="0 0 0" rpy="${pi / 2.0} 0 0" />
+            </collision>
+            <xacro:cylinder_inertia mass="1.0" radius="${wheel_radius}" height="${wheel_length}"
+                xyz="0 0 0" rpy="${pi / 2.0} 0 0" />
         </link>
-        <xacro:cylinder_inertia mass="1.0" radius="${wheel_radius}" height="${wheel_length}"
-            xyz="0 0 0" rpy="${pi / 2.0} 0 0" />
     </xacro:macro>
     <xacro:wheel_link prefix="right" />
@@ -41,4 +53,10 @@
             <material name="grey" />
         </visual>
+        <collision>
+            <geometry>
+                <sphere radius="${wheel_radius / 2.0}" />
+            </geometry>
+            <origin xyz="0 0 0" rpy="0 0 0" />
+        </collision>
         <xacro:sphere_inertia mass="0.5" radius="${wheel_radius / 2.0}" xyz="0 0 0" rpy="0 0 0" />
     </link>

Commit message: add robot arm

File: src/my_robot_description/urdf/common_properties.xacro (robot description, xacro)
@@ -6,4 +6,10 @@
     <material name="grey">
         <color rgba="0.5 0.5 0.5 1" />
+    </material>
+    <material name="orange">
+        <color rgba="1 0.5 0 1" />
+    </material>
+    <material name="yellow">
+        <color rgba="1 1 0 1" />
     </material>
     <xacro:macro name="box_inertia" params="mass length width height xyz rpy">
