Commit message: combine robots

File: src/my_robot_description/urdf/arm_gazebo.xacro (robot description, xacro)
@@ -17,5 +17,5 @@
 			<!-- Name of joints in the model whose states will be published. -->
 			<joint_name>arm_base_forearm_joint</joint_name>
-			<joint_name>foream_hand_joint</joint_name>
+			<joint_name>forearm_hand_joint</joint_name>
 		</plugin>
 	</gazebo>

File: src/my_robot_description/urdf/my_robot.urdf.xacro (robot description, xacro)
@@ -5,3 +5,11 @@
     <xacro:include filename="mobile_base_gazebo.xacro" />
     <xacro:include filename="camera.xacro" />
+    <!-- Adding robot arm -->
+    <xacro:include filename="arm.xacro" />
+    <xacro:include filename="arm_gazebo.xacro" />
+    <joint name="mobile_base_arm_joint" type="fixed">
+        <parent link="base_link" />
+        <child link="arm_base_link" />
+        <origin xyz="${base_length/4} 0 ${base_height}" rpy="0 0 0" />
+    </joint>
 </robot>
